File: new_job.kicad_pcb (KiCad board)
At the start: 2 copper layers, 140 x 70 mm, 248 parts, among them J1 PWM_OUT, J10 PWM_OUT, J11 AC_OUT, J12 AC_OUT, J13 AC_OUT, J14 AC_OUT, J15 SPK, J16 LEVEL_LOW, J17 LEVEL_HIGH, J18 LEVEL_HIGH, J19 VIN, J2 PWM_OUT, J20 Conn_01x04_Pin, J21 IR, J3 PWM_OUT, J4 PWM_OUT, J5 PWM_OUT, J6 PWM_OUT, J7 PWM_OUT, J8 PWM_OUT, J9 Conn_01x10_Pin, K1 SANYOU_SRD_Form_C, K2 SANYOU_SRD_Form_C, K3 SANYOU_SRD_Form_C, K4 SANYOU_SRD_Form_C, Q1 IRFR220, Q10 2N7002H, Q11 2N7002H, Q12 2N7002H, Q13 2N7002H, Q2 IRFR220, Q3 IRFR220, Q4 IRFR220, Q5 IRFR220, Q6 IRFR220, Q7 IRFR220, Q8 IRFR220, Q9 IRFR220, SW1 SW_Push, SW2 SW_Push, SW3 SW_Push, SW4 SW_Push, SW5 SW_Push, U1 STM32F030C6Tx, U10 TLP152, U11 DFR0299, U12 RY9130, U13 RY9130, U2 TLP152, U3 TLP152, U4 TLP152, U5 TLP152, U6 TLP152, U7 TLP152, U8 TLP152, U9 TLP152, Y1 8Mhz, Y2 32.768KHz

Commit message: PCB improoved
Parts:
- removed C37, C38, C49, C50, C62, C63, C72, C73, C84, C85: 1uF, Capacitor_SMD:C_0402_1005Metric
- removed C52: 4.7uF, Capacitor_SMD:C_0201_0603Metric
- removed C53, C64, C65, C74, C86: 100nF, Capacitor_SMD:C_0402_1005Metric
- removed F1: 630mA, Fuse:Fuse_0603_1608Metric
- C24, C33, C34, C35, C51, C59, C60, C69, C7, C70, C81, C82: footprint Capacitor_SMD:C_0201_0603Metric -> Capacitor_SMD:C_0603_1608Metric
- C29: value 470uF -> 100nF; footprint Capacitor_SMD:CP_Elec_10x10.5 -> Capacitor_SMD:C_0402_1005Metric
- J16, J17, J18: footprint Connector_Molex:Molex_SL_171971-0002_1x02_P2.54mm_Vertical -> Connector_PinHeader_2.54mm:PinHeader_1x02_P2.54mm_Vertical
- moved J9 375.2 mm to (217.7, 70.5), turned to -90 degrees
- moved L1 347.3 mm to (193.0, 86.0), turned to -90 degrees
- moved D9 338.5 mm to (216.0, 115.0)
- moved C28 338.3 mm to (214.7, 85.0)
- moved C27 335.7 mm to (214.7, 96.5)
- moved C26 334.7 mm to (214.7, 108.0)
- moved C42 328.4 mm to (206.0, 75.5), turned to 90 degrees
- moved C39 324.8 mm to (208.0, 88.5), turned to -90 degrees
- moved D5 322.7 mm to (125.5, 91.0), turned to 180 degrees
- moved C40 322.5 mm to (208.0, 100.0), turned to -90 degrees
- moved D4 322.1 mm to (125.5, 85.0), turned to 0 degrees
- moved C29 321.5 mm to (194.0, 77.0), turned to 180 degrees
- moved C41 320.4 mm to (208.0, 111.5), turned to -90 degrees
- moved D3 318.1 mm to (133.0, 85.0), turned to 0 degrees
- moved C45 316.2 mm to (196.0, 86.0), turned to 90 degrees
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Connections:
- D9 pad 1: Net-(D9-K) -> +12V
- J19 pad 1: Net-(D9-K) -> +12V
Routing:
- net /SWCLK: track 7.63 -> 5.98 mm
- net /SWDIO: track 10.5 -> 8.82 mm
Other:
- board size 140 x 70 mm -> 175 x 57 mm

Commit message: production ready
Parts:
- removed C10, C11, C32: 10uF, Capacitor_SMD:C_0805_2012Metric
- removed C34, C35: 4.7uF, Capacitor_SMD:C_0603_1608Metric
- removed R82: 10k, Resistor_SMD:R_0402_1005Metric
- J11, J12, J13, J14: footprint Connector_Molex:Molex_SL_171971-0002_1x02_P2.54mm_Vertical -> TerminalBlock_RND:TerminalBlock_RND_205-00067_1x02_P7.50mm_Horizontal
- moved C36 334.1 mm to (207.5, 76.3), turned to 90 degrees
- moved C30 316.2 mm to (213.8, 78.3)
- moved C31 314.9 mm to (210.9, 76.3), turned to 90 degrees
- moved R44 289.6 mm to (214.0, 74.4), turned to 90 degrees
- moved R43 288.2 mm to (212.8, 74.4), turned to 90 degrees
- moved C3 282.5 mm to (159.6, 93.2), turned to -90 degrees
- moved C4 280.9 mm to (153.2, 80.7)
- moved C6 279.8 mm to (151.2, 80.4), turned to -90 degrees
- moved C33 273.6 mm to (208.9, 76.3), turned to 90 degrees
- moved C94 261.7 mm to (118.2, 120.7), turned to 180 degrees
- moved C93 261.3 mm to (118.2, 119.7), turned to 180 degrees
- moved C92 261.0 mm to (118.2, 118.7), turned to 180 degrees
- moved C5 257.5 mm to (147.7, 79.0), turned to 90 degrees
- moved C12 251.0 mm to (121.1, 86.3), turned to -90 degrees
- moved R2 234.9 mm to (151.1, 76.5), turned to 180 degrees
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Connections:
- net Net-(J1-Pin_2) renamed /PWM_OUT_8
- net Net-(J2-Pin_2) renamed /PWM_OUT_7
- net Net-(J3-Pin_2) renamed /PWM_OUT_6
- net Net-(J4-Pin_2) renamed /PWM_OUT_5
- net Net-(J5-Pin_2) renamed /PWM_OUT_3
- net Net-(J6-Pin_2) renamed /PWM_OUT_2
- net Net-(J7-Pin_2) renamed /PWM_OUT_1
- net Net-(J8-Pin_2) renamed /PWM_OUT_4
- net Net-(U12-SW) renamed /L_OUT
- net Net-(U13-SW) renamed /L_OUT_5V
- J10 pad 2: Net-(J10-Pin_2) -> /DC_OUT
- J15 pad 1: /SPK_DN -> /SPK_DP
- J15 pad 2: /SPK_DP -> /SPK_DN
- J9 pad 1: /SCL -> /GPIO4
- J9 pad 10: /GPIO4 -> GND
- J9 pad 3: /SPI_CS -> /SCL
- J9 pad 4: /SPI_SCK -> /SPI_CS
- J9 pad 5: /SPI_MISO -> /SPI_SCK
- J9 pad 6: /SPI_MOSI -> /SPI_MISO
- J9 pad 7: unconnected-(J9-Pin_7-Pad7) -> /SPI_MOSI
- J9 pad 8: /GPIO2 -> /GPIO3
- J9 pad 9: /GPIO3 -> /GPIO2
- K1 pad 1: Net-(J13-Pin_2) -> Net-(J11-Pin_1)
- K1 pad 3: Net-(J13-Pin_1) -> Net-(J11-Pin_2)
- K2 pad 1: Net-(J12-Pin_2) -> Net-(J12-Pin_1)
- K2 pad 3: Net-(J12-Pin_1) -> Net-(J12-Pin_2)
- K3 pad 1: Net-(J14-Pin_2) -> Net-(J13-Pin_1)
- K3 pad 3: Net-(J14-Pin_1) -> Net-(J13-Pin_2)
- K4 pad 1: Net-(J11-Pin_2) -> Net-(J14-Pin_1)
- K4 pad 3: Net-(J11-Pin_1) -> Net-(J14-Pin_2)
- Q6 pad 2: Net-(J10-Pin_2) -> /DC_OUT
- R51 pad 1: /DC_OUT -> /DC_OUT_CMD
- U1 pad 15: /GPIO2 -> /DC_OUT_CMD
- U1 pad 16: /PWM3 -> /PWM7
- U1 pad 17: /PWM4 -> /PWM6
- U1 pad 18: /PWM1 -> /PWM5
- U1 pad 19: /PWM2 -> /PWM8
- U1 pad 2: /RELAY2 -> /RELAY1
- U1 pad 29: /PWM5 -> /PWM2
- U1 pad 30: /PWM6 -> /PWM1
- U1 pad 31: /PWM7 -> /PWM3
- U1 pad 32: /PWM8 -> /PWM4
- U1 pad 33: /RELAY1 -> /RELAY2
- U1 pad 39: /DC_OUT -> /GPIO2
- U1 pad 40: /BTN1 -> /BTN3
- U1 pad 42: /BTN3 -> /BTN1
- U13 pad 4: Net-(U13-EN) -> +12V
Routing:
- net +12V: track 0.00 -> 274.0 mm, vias 0 -> 54
- net +3.3V: track 0.00 -> 108.0 mm, vias 0 -> 45
- net /RELAY3: track 0.00 -> 98.5 mm, vias 0 -> 2
- net /RELAY1: track 0.00 -> 93.5 mm, vias 0 -> 2
- net /RELAY2: track 0.00 -> 81.6 mm, vias 0 -> 2
- net /RELAY4: track 0.00 -> 80.7 mm, vias 0 -> 2
- net /GPIO4: track 0.00 -> 80.6 mm, vias 0 -> 1
- net /IR_IN: track 0.00 -> 78.5 mm, vias 0 -> 2
- net /SDA: track 0.00 -> 76.4 mm, vias 0 -> 1
- net /SCL: track 0.00 -> 75.2 mm, vias 0 -> 1
- net /MCU_RX: track 0.00 -> 73.7 mm
- net /SPI_CS: track 0.00 -> 62.2 mm, vias 0 -> 1
- net /MCU_TX: track 0.00 -> 59.3 mm
- net /SPI_SCK: track 0.00 -> 57.5 mm, vias 0 -> 1
- net /SPI_MISO: track 0.00 -> 53.2 mm, vias 0 -> 1
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- added copper zone on F.Cu, net +12V
- added copper zone on In2.Cu, net +12V
- added copper zone on F.Cu, net +3.3V
- added copper zone on In2.Cu, net +3.3V
- added copper zone on F.Cu, net +5V
- added copper zone on In2.Cu, net +5V
- added copper zone on F.Cu, net /DC_OUT
- added copper zone on F.Cu, net /L_OUT
- added copper zone on F.Cu, net /L_OUT_5V
- added copper zone on F.Cu, net /PWM_OUT_1
- added copper zone on F.Cu, net /PWM_OUT_2
- added copper zone on F.Cu, net /PWM_OUT_3
- added copper zone on F.Cu, net /PWM_OUT_4
- added copper zone on F.Cu, net /PWM_OUT_5
- added copper zone on F.Cu, net /PWM_OUT_6
- added copper zone on F.Cu, net /PWM_OUT_7
- added copper zone on F.Cu, net /PWM_OUT_8
- added copper zone on B.Cu, net GND
- added copper zone on F.Cu, net GND
- added copper zone on In1.Cu, net GND
- added copper zone on In2.Cu, net GND
Other:
- board size 175 x 57 mm -> 175 x 59 mm
- copper layers 2 -> 4
- board text added: "Y O R O Z U Y A design studio"
- board text added: "bunu oxuyursansa qarantiyan bitdi))"
- board text added: "product of Kaminci.az"
